File: hardware/motors.kicad_sch (KiCad schematic)
At the start: 11 parts, among them J2 JST_PH_01x02, J3 JST_XH_01x02, J4 JST_XH_01x02, U3 DRV8212, U4 DRV8212

Commit message: Fixed motor driver grounding
Made new footprint with smaller thermal vias for less solder wicking.
Added more vias in ground puddle.
Parts:
- U3, U4: footprint Package_SON:WSON-8-1EP_2x2mm_P0.5mm_EP0.9x1.6mm_ThermalVias -> heli-footprints:WSON-8-1EP_2x2mm_P0.5mm_EP0.9x1.6mm_ThermalVias
Changed lines of the file:
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@@
 			)
 		)
-		(property "Footprint" "Package_SON:WSON-8-1EP_2x2mm_P0.5mm_EP0.9x1.6mm_ThermalVias"
+		(property "Footprint" "heli-footprints:WSON-8-1EP_2x2mm_P0.5mm_EP0.9x1.6mm_ThermalVias"
 			(at 191.77 125.73 0)
 			(effects
@@
 			)
 		)
-		(property "Footprint" "Package_SON:WSON-8-1EP_2x2mm_P0.5mm_EP0.9x1.6mm_ThermalVias"
+		(property "Footprint" "heli-footprints:WSON-8-1EP_2x2mm_P0.5mm_EP0.9x1.6mm_ThermalVias"
 			(at 76.2 129.54 0)
 			(effects
