File: hardware/heli_avionics.kicad_pcb (KiCad board)
At the start: 4 copper layers, 65.5 x 39 mm, 76 parts, among them J1 Pin_Header_2x3, J10 Pin_Header_1x1, J2 JST_PH_01x02, J3 JST_XH_01x02, J4 JST_XH_01x02, J5 JST_PH_01x03, J6 Conn_01x01, J7 JST_1.25mm, J8 Conn_01x01, J9 Pin_Header_1x2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

Commit message: Add some soldermask expansion on motor drivers
Parts:
- U5: value BMP390L -> XDCR_BMP390L
Changed lines of the file:
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@@
 			)
 		)
-		(property "Value" "BMP390L"
+		(property "Value" "XDCR_BMP390L"
 			(at 1.1884 1.5532 0)
 			(layer "F.Fab")
@@
 		(sheetname "Pressure sensor")
 		(sheetfile "sensors.kicad_sch")
-		(solder_mask_margin 0.038)
+		(solder_mask_margin 0.0254)
 		(attr smd)
 		(fp_line
@@
 		(sheetname "Motor Drivers")
 		(sheetfile "motors.kicad_sch")
+		(solder_mask_margin 0.0254)
 		(fp_line
 			(start -1.01 -1.14)
@@
 		(sheetname "Motor Drivers")
 		(sheetfile "motors.kicad_sch")
+		(solder_mask_margin 0.0254)
 		(fp_line
 			(start -1.01 -1.14)
@@
 		(sheetname "Motor Drivers")
 		(sheetfile "motors.kicad_sch")
+		(solder_mask_margin 0.0254)
 		(fp_line
 			(start -1.01 -1.14)
